Commit message: added moving camera

File: annin_ar4_description/urdf/ar_gazebo.urdf.xacro (robot description, xacro)
@@ -37,4 +37,33 @@
     tf_prefix="$(arg tf_prefix)"
   />
+  <!-- Camera link fixed to end-effector -->
+  <link name="$(arg tf_prefix)ee_camera_link">
+    <inertial>
+      <origin xyz="0 0 0" rpy="0 0 0"/>
+      <mass value="0.1"/>
+      <inertia ixx="0.0001" ixy="0" ixz="0" iyy="0.0001" iyz="0" izz="0.0001"/>
+    </inertial>
+    <visual>
+      <origin xyz="0 0 0" rpy="0 0 0"/>
+      <geometry>
+        <box size="0.02 0.02 0.02"/>
+      </geometry>
+      <material name="camera_material">
+        <color rgba="0.2 0.2 0.8 1"/>
+      </material>
+    </visual>
+    <collision>
+      <origin xyz="0 0 0" rpy="0 0 0"/>
+      <geometry>
+        <box size="0.02 0.02 0.02"/>
+      </geometry>
+    </collision>
+  </link>
+  <joint name="$(arg tf_prefix)ee_camera_fixed" type="fixed">
+    <parent link="$(arg tf_prefix)ee_link"/>
+    <child link="$(arg tf_prefix)ee_camera_link"/>
+    <!-- Adjust pose to your mount; z offset puts it ahead of flange -->
+    <origin xyz="0 0 0.02" rpy="0 0 0"/>
+  </joint>
   <gazebo reference="world" />
   <gazebo>
@@ -46,3 +75,25 @@
     </plugin>
   </gazebo>
+  <!-- Gazebo Sim camera sensor attached to ee_camera_link -->
+  <gazebo reference="$(arg tf_prefix)ee_camera_link">
+    <sensor type="camera" name="ee_camera_sensor">
+      <pose>0 0 0 0 0 0</pose>
+      <camera>
+        <horizontal_fov>1.047</horizontal_fov>
+        <image>
+          <width>320</width>
+          <height>240</height>
+          <format>R8G8B8</format>
+        </image>
+        <clip>
+          <near>0.1</near>
+          <far>100</far>
+        </clip>
+      </camera>
+      <always_on>1</always_on>
+      <update_rate>30</update_rate>
+      <visualize>true</visualize>
+      <topic>rgb_camera_moving/image</topic>
+    </sensor>
+  </gazebo>
 </robot>

Commit message: improved coordinate frame of robot

File: annin_ar4_description/urdf/ar_gazebo.urdf.xacro (robot description, xacro)
@@ -14,5 +14,5 @@
     robot_parameters_file="$(find annin_ar4_description)/config/$(arg ar_model).yaml"
   >
-    <origin xyz="0 0 0" rpy="0 0 0" />
+    <origin xyz="0 0 0" rpy="0 0 4.712" />
   </xacro:ar_robot>
   <xacro:ar_gripper

Commit message: working on coordinate transform bug

File: annin_ar4_description/urdf/ar_gazebo.urdf.xacro (robot description, xacro)
@@ -8,4 +8,5 @@
   <xacro:arg name="tf_prefix" default="" />
   <xacro:arg name="namespace" default="" />
+  <xacro:arg name="base_yaw" default="4.712" />
   <link name="world" />
   <xacro:ar_robot
@@ -14,5 +15,5 @@
     robot_parameters_file="$(find annin_ar4_description)/config/$(arg ar_model).yaml"
   >
-    <origin xyz="0 0 0" rpy="0 0 4.712" />
+    <origin xyz="0 0 0" rpy="0 0 $(arg base_yaw)" />
   </xacro:ar_robot>
   <xacro:ar_gripper
@@ -79,5 +80,5 @@
     <sensor type="rgbd_camera" name="ee_rgbd_sensor">
       <!-- Identity pose - camera frame aligned with ee_camera_link frame -->
-      <pose>0 0 0 0 0 0</pose>
+      <pose>0 0 0 1.57 -1.57 0</pose>
       <camera>
         <horizontal_fov>1.047</horizontal_fov>
