Commit message: fixed minor bug

File: annin_ar4_description/urdf/ar_macro.xacro (robot description, xacro)
@@ -8,7 +8,16 @@
   ">
     <xacro:property name="robot_parameters" value="${xacro.load_yaml(robot_parameters_file)}"/>
+    <!-- Apply external rotation/translation to a mount link, keep internal joints untouched -->
+    <link name="${tf_prefix}base_mount" />
+    <!-- Parent -> base_mount with provided origin (rotation/translation) -->
     <joint name="${tf_prefix}base_joint" type="fixed">
       <xacro:insert_block name="origin" />
       <parent link="${parent}"/>
+      <child link="${tf_prefix}base_mount" />
+    </joint>
+    <!-- base_mount -> base_link identity transform -->
+    <joint name="${tf_prefix}base_mount_to_base" type="fixed">
+      <origin rpy="0 0 0" xyz="0 0 0" />
+      <parent link="${tf_prefix}base_mount" />
       <child link="${tf_prefix}base_link" />
     </joint>

Commit message: up to date

File: annin_ar4_description/urdf/ar_macro.xacro (robot description, xacro)
@@ -203,5 +203,5 @@
     </link>
     <joint name="${tf_prefix}joint_5" type="revolute">
-      <origin rpy="${pi} 0 -1.5708" xyz="0 0 -0.22263"/>
+      <origin rpy="${3*pi/2} 0 -1.5708" xyz="0 0 -0.22263"/>
       <parent link="${tf_prefix}link_4"/>
       <child link="${tf_prefix}link_5"/>
