Commit message: working on frame transform

File: annin_ar4_description/urdf/ar.urdf.xacro (robot description, xacro)
@@ -3,4 +3,5 @@
   <xacro:arg name="tf_prefix" default="" />
   <xacro:arg name="include_gripper" default="true"/>
+  <xacro:arg name="base_yaw" default="4.712"/> <!-- Add this line -->
   <xacro:include filename="$(find annin_ar4_description)/urdf/ar_macro.xacro"/>
   <link name="world" />
@@ -10,5 +11,5 @@
     robot_parameters_file="$(find annin_ar4_description)/config/$(arg ar_model).yaml"
   >
-    <origin xyz="0 0 0" rpy="0 0 0" />
+    <origin xyz="0 0 0" rpy="0 0 $(arg base_yaw)" /> <!-- Change here -->
   </xacro:ar_robot>
   <xacro:if value="$(arg include_gripper)">

File: annin_ar4_moveit_config/urdf/fake_ar.urdf.xacro (robot description, xacro)
@@ -1,9 +1,10 @@
 <?xml version="1.0"?>
 <robot xmlns:xacro="http://wiki.ros.org/xacro" name="$(arg ar_model)">
+  <xacro:arg name="tf_prefix" default="" />
+  <xacro:arg name="base_yaw" default="4.712"/> <!-- Add this line -->
   <xacro:include filename="$(find annin_ar4_description)/urdf/ar_macro.xacro"/>
   <xacro:include filename="$(find annin_ar4_description)/urdf/ar_gripper_macro.xacro"/>
   <xacro:include filename="$(find annin_ar4_description)/urdf/ar.ros2_control.xacro"/>
   <xacro:include filename="$(find annin_ar4_description)/urdf/ar_gripper.ros2_control.xacro"/>
-  <xacro:arg name="tf_prefix" default="" />
   <link name="world" />
   <xacro:ar_robot
@@ -12,5 +13,5 @@
     robot_parameters_file="$(find annin_ar4_description)/config/$(arg ar_model).yaml"
   >
-    <origin xyz="0 0 0" rpy="0 0 0" />
+    <origin xyz="0 0 0" rpy="0 0 $(arg base_yaw)" /> <!-- Change here -->
   </xacro:ar_robot>
   <xacro:ar_gripper

Commit message: added visualized camera

File: annin_ar4_description/urdf/ar.urdf.xacro (robot description, xacro)
@@ -20,3 +20,17 @@
     />
   </xacro:if>
+  <!-- Camera mount frame (matches Gazebo URDF so ee_camera_link TF exists) -->
+  <link name="$(arg tf_prefix)ee_camera_link">
+    <inertial>
+      <origin xyz="0 0 0" rpy="0 0 0"/>
+      <mass value="0.1"/>
+      <inertia ixx="0.0001" ixy="0" ixz="0" iyy="0.0001" iyz="0" izz="0.0001"/>
+    </inertial>
+  </link>
+  <joint name="$(arg tf_prefix)ee_camera_fixed" type="fixed">
+    <parent link="$(arg tf_prefix)ee_link"/>
+    <child link="$(arg tf_prefix)ee_camera_link"/>
+    <!-- Adjust xyz/rpy to match your physical camera mount -->
+    <origin xyz="0 0 0.02" rpy="0 0 0"/>
+  </joint>
 </robot>

File: annin_ar4_description/urdf/ar_gazebo.urdf.xacro (robot description, xacro)
@@ -48,5 +48,5 @@
       <origin xyz="0 0 0" rpy="0 0 0"/>
       <geometry>
-        <box size="0.02 0.02 0.02"/>
+        <box size="0.05 0.03 0.03"/>
       </geometry>
       <material name="camera_material">
@@ -54,8 +54,17 @@
       </material>
     </visual>
+    <visual>
+      <origin xyz="0 0 0.025" rpy="0 0 0"/>
+      <geometry>
+        <cylinder radius="0.012" length="0.02"/>
+      </geometry>
+      <material name="camera_lens">
+        <color rgba="0.1 0.1 0.1 1"/>
+      </material>
+    </visual>
     <collision>
       <origin xyz="0 0 0" rpy="0 0 0"/>
       <geometry>
-        <box size="0.02 0.02 0.02"/>
+        <box size="0.05 0.03 0.03"/>
       </geometry>
     </collision>
@@ -64,6 +73,6 @@
     <parent link="$(arg tf_prefix)ee_link"/>
     <child link="$(arg tf_prefix)ee_camera_link"/>
-    <!-- Adjust pose to your mount; z offset puts it ahead of flange -->
-    <origin xyz="0 0 0.02" rpy="0 0 0"/>
+    <!-- Offset sideways (X) to clear the gripper -->
+    <origin xyz="0.05 0 0.02" rpy="0 0 0"/>
   </joint>
   <gazebo reference="world" />

File: annin_ar4_driver/urdf/ar.urdf.xacro (robot description, xacro)
@@ -41,3 +41,17 @@
     />
   </xacro:if>
+  <!-- Camera mount frame (so ee_camera_link TF exists for ArUco detection) -->
+  <link name="$(arg tf_prefix)ee_camera_link">
+    <inertial>
+      <origin xyz="0 0 0" rpy="0 0 0"/>
+      <mass value="0.1"/>
+      <inertia ixx="0.0001" ixy="0" ixz="0" iyy="0.0001" iyz="0" izz="0.0001"/>
+    </inertial>
+  </link>
+  <joint name="$(arg tf_prefix)ee_camera_fixed" type="fixed">
+    <parent link="$(arg tf_prefix)ee_link"/>
+    <child link="$(arg tf_prefix)ee_camera_link"/>
+    <!-- Adjust xyz/rpy to match your physical camera mount -->
+    <origin xyz="0 0 0.02" rpy="0 0 0"/>
+  </joint>
 </robot>

Commit message: just checking

File: annin_ar4_description/urdf/ar.urdf.xacro (robot description, xacro)
@@ -32,5 +32,5 @@
     <child link="$(arg tf_prefix)ee_camera_link"/>
     <!-- Adjust xyz/rpy to match your physical camera mount -->
-    <origin xyz="0 0 0.02" rpy="0 0 0"/>
+    <origin xyz="-0.05 0 0.02" rpy="0 0 0"/>
   </joint>
 </robot>

File: annin_ar4_description/urdf/ar_gazebo.urdf.xacro (robot description, xacro)
@@ -74,5 +74,5 @@
     <child link="$(arg tf_prefix)ee_camera_link"/>
     <!-- Offset sideways (X) to clear the gripper -->
-    <origin xyz="0.05 0 0.02" rpy="0 0 0"/>
+    <origin xyz="-0.05 0 0.02" rpy="0 0 0"/>
   </joint>
   <gazebo reference="world" />

Commit message: added camera offsets

File: annin_ar4_description/urdf/ar.urdf.xacro (robot description, xacro)
@@ -32,5 +32,5 @@
     <child link="$(arg tf_prefix)ee_camera_link"/>
     <!-- Adjust xyz/rpy to match your physical camera mount -->
-    <origin xyz="-0.05 0 0.02" rpy="0 0 0"/>
+    <origin xyz="-0.06 0 0.04" rpy="0 0 1.5708"/>
   </joint>
 </robot>

File: annin_ar4_driver/urdf/ar.urdf.xacro (robot description, xacro)
@@ -53,5 +53,5 @@
     <child link="$(arg tf_prefix)ee_camera_link"/>
     <!-- Adjust xyz/rpy to match your physical camera mount -->
-    <origin xyz="0 0 0.02" rpy="0 0 0"/>
+    <origin xyz="-0.06 0 0.04" rpy="0 0 1.5708"/>
   </joint>
 </robot>
