Commit message: a bug fix

File: annin_ar4_description/urdf/ar.ros2_control.xacro (robot description, xacro)
@@ -10,5 +10,12 @@
     driver_parameters_file
     tf_prefix
+    j1_home:=0.0 j2_home:=0.0 j3_home:=0.0 j4_home:=0.0 j5_home:=0.0 j6_home:=0.0
   ">
+    <!-- j*_home feeds the position state interfaces' initial_value below, i.e.
+         the pose a SIMULATED arm starts at. Defaults are zeros so the real
+         driver's behaviour is unchanged (it reports actual encoder positions and
+         ignores initial_value); ar_gazebo.urdf.xacro passes the 'home'
+         group_state from annin_ar4_moveit_config/srdf/ar_macro.srdf.xacro, so
+         the sim spawns exactly where RViz's home button sends the arm. -->
     <xacro:property name="robot_parameters"
       value="${xacro.load_yaml(robot_parameters_file)}"/>
@@ -34,5 +41,5 @@
         <command_interface name="velocity" />
         <state_interface name="position">
-          <param name="initial_value">0.0</param>
+          <param name="initial_value">${j1_home}</param>
         </state_interface>
         <state_interface name="velocity">
@@ -48,5 +55,5 @@
         <command_interface name="velocity" />
         <state_interface name="position">
-          <param name="initial_value">0.0</param>
+          <param name="initial_value">${j2_home}</param>
         </state_interface>
         <state_interface name="velocity">
@@ -62,5 +69,5 @@
         <command_interface name="velocity" />
         <state_interface name="position">
-          <param name="initial_value">0.0</param>
+          <param name="initial_value">${j3_home}</param>
         </state_interface>
         <state_interface name="velocity">
@@ -76,5 +83,5 @@
         <command_interface name="velocity" />
         <state_interface name="position">
-          <param name="initial_value">0.0</param>
+          <param name="initial_value">${j4_home}</param>
         </state_interface>
         <state_interface name="velocity">
@@ -90,5 +97,5 @@
         <command_interface name="velocity" />
         <state_interface name="position">
-          <param name="initial_value">0.0</param>
+          <param name="initial_value">${j5_home}</param>
         </state_interface>
         <state_interface name="velocity">
@@ -104,5 +111,5 @@
         <command_interface name="velocity" />
         <state_interface name="position">
-          <param name="initial_value">0.0</param>
+          <param name="initial_value">${j6_home}</param>
         </state_interface>
         <state_interface name="velocity">

File: annin_ar4_description/urdf/ar_gazebo.urdf.xacro (robot description, xacro)
@@ -21,4 +21,8 @@
     parent="$(arg tf_prefix)ee_link"
   />
+  <!-- j*_home: the pose gz spawns the arm at. MUST match the 'home' group_state
+       in annin_ar4_moveit_config/srdf/ar_macro.srdf.xacro (the all-zero pose
+       lifted 5 cm, so a gripper closing at home clears the floor) — otherwise
+       the arm spawns somewhere RViz's home button will not return it to. -->
   <xacro:ar_ros2_control
     ar_model="$(arg ar_model)"
@@ -30,4 +34,6 @@
     driver_parameters_file="$(find annin_ar4_driver)/config/driver.yaml"
     tf_prefix="$(arg tf_prefix)"
+    j1_home="0.0" j2_home="0.0187" j3_home="-0.2455"
+    j4_home="0.0" j5_home="0.2268" j6_home="0.0"
   />
   <xacro:ar_gripper_ros2_control

File: annin_ar4_moveit_config/srdf/ar_macro.srdf.xacro (robot description, xacro)
@@ -15,10 +15,18 @@
       <joint name="${tf_prefix}ee_joint"/>
     </group>
+    <!-- Home: the all-zero pose lifted 5 cm in +z, with x/y and the tool axis
+         unchanged (zeros put link_6 at z=0.434 m, tool pointing straight down).
+         joint_2/joint_5 pitch by opposite amounts so the tool keeps pointing
+         down, joint_3 takes up the lateral drift. The clearance matters because
+         a gripper closes at home without the arm moving, and the planner has no
+         way to back the arm off. Keep in sync with the initial_value params in
+         annin_ar4_description/urdf/ar_gazebo.urdf.xacro so the sim spawns here,
+         and note ar4Automating3DPrinter's go_home reads THIS state at runtime. -->
     <group_state name="home" group="ar_manipulator">
       <joint name="${tf_prefix}joint_1" value="0" />
-      <joint name="${tf_prefix}joint_2" value="0" />
-      <joint name="${tf_prefix}joint_3" value="0" />
+      <joint name="${tf_prefix}joint_2" value="0.0187" />
+      <joint name="${tf_prefix}joint_3" value="-0.2455" />
       <joint name="${tf_prefix}joint_4" value="0" />
-      <joint name="${tf_prefix}joint_5" value="0" />
+      <joint name="${tf_prefix}joint_5" value="0.2268" />
       <joint name="${tf_prefix}joint_6" value="0" />
     </group_state>

File: annin_ar4_moveit_config/urdf/fake_ar.urdf.xacro (robot description, xacro)
@@ -19,4 +19,6 @@
     parent="$(arg tf_prefix)ee_link"
   />
+  <!-- j*_home starts the mock robot at the SRDF 'home' group_state, like the gz
+       spawn — see annin_ar4_moveit_config/srdf/ar_macro.srdf.xacro -->
   <xacro:ar_ros2_control
     ar_model="$(arg ar_model)"
@@ -28,4 +30,6 @@
     driver_parameters_file="$(find annin_ar4_driver)/config/driver.yaml"
     tf_prefix="$(arg tf_prefix)"
+    j1_home="0.0" j2_home="0.0187" j3_home="-0.2455"
+    j4_home="0.0" j5_home="0.2268" j6_home="0.0"
   />
   <xacro:ar_gripper_ros2_control
